File: Cordonatrice F.lli Verna.kicad_pcb (KiCad board)
At the start: 2 copper layers, 6 parts, among them P1 CONN_01X10, P2 CONN_01X10, U2 TXS0108EPW

Commit message: correzione schema corretto
Parts:
- removed C1, C2: 0.1uF, Capacitor_SMD:C_0805_2012Metric_Pad1.18x1.45mm_HandSolder
- removed P1, P2: CONN_01X10, Connector_PinHeader_2.54mm:PinHeader_1x10_P2.54mm_Vertical
- added C3: 100nF_Ceramic, Capacitor_THT:C_Disc_D5.0mm_W2.5mm_P2.50mm, F.Cu at (157.5, 118.0)
- added C4: 100nF_Ceramic, Capacitor_THT:C_Disc_D5.0mm_W2.5mm_P2.50mm, F.Cu at (157.5, 122.0)
- added C5: 22uF_50V, Capacitor_THT:CP_Radial_D5.0mm_P2.00mm, F.Cu at (157.8, 106.1)
- added C6: 22uF_50V, Capacitor_THT:CP_Radial_D5.0mm_P2.00mm, F.Cu at (157.8, 112.7)
- added J1: Screw_Terminal_3_P5.00mm, TerminalBlock_Phoenix:TerminalBlock_Phoenix_PT-1,5-3-5.0-H_1x03_P5.00mm_Horizontal, F.Cu at (91.0, 40.6)
- added J10: Screw_Terminal_2_P5.00mm, TerminalBlock_Phoenix:TerminalBlock_Phoenix_PT-1,5-2-5.0-H_1x02_P5.00mm_Horizontal, F.Cu at (108.1, 51.9)
- added J11: Screw_Terminal_2_P5.00mm, TerminalBlock_Phoenix:TerminalBlock_Phoenix_PT-1,5-2-5.0-H_1x02_P5.00mm_Horizontal, F.Cu at (108.1, 63.2)
- added J12: Screw_Terminal_4_P5.00mm, TerminalBlock_Phoenix:TerminalBlock_Phoenix_PT-1,5-4-5.0-H_1x04_P5.00mm_Horizontal, F.Cu at (147.3, 96.5)
- added J13: Screw_Terminal_2_P5.00mm, TerminalBlock_Phoenix:TerminalBlock_Phoenix_PT-1,5-2-5.0-H_1x02_P5.00mm_Horizontal, F.Cu at (108.1, 74.5)
- added J14: Screw_Terminal_2_P5.00mm, TerminalBlock_Phoenix:TerminalBlock_Phoenix_PT-1,5-2-5.0-H_1x02_P5.00mm_Horizontal, F.Cu at (108.1, 85.8)
- added J2: Screw_Terminal_3_P5.00mm, TerminalBlock_Phoenix:TerminalBlock_Phoenix_PT-1,5-3-5.0-H_1x03_P5.00mm_Horizontal, F.Cu at (91.0, 51.9)
- added J3: Screw_Terminal_3_P5.00mm, TerminalBlock_Phoenix:TerminalBlock_Phoenix_PT-1,5-3-5.0-H_1x03_P5.00mm_Horizontal, F.Cu at (91.0, 63.2)
- added J4: Screw_Terminal_3_P5.00mm, TerminalBlock_Phoenix:TerminalBlock_Phoenix_PT-1,5-3-5.0-H_1x03_P5.00mm_Horizontal, F.Cu at (91.0, 74.5)
- added J5: Screw_Terminal_3_P5.00mm, TerminalBlock_Phoenix:TerminalBlock_Phoenix_PT-1,5-3-5.0-H_1x03_P5.00mm_Horizontal, F.Cu at (91.0, 85.8)
- added J6: Screw_Terminal_3_P5.00mm, TerminalBlock_Phoenix:TerminalBlock_Phoenix_PT-1,5-3-5.0-H_1x03_P5.00mm_Horizontal, F.Cu at (91.0, 97.2)
- added J7: Screw_Terminal_3_P5.00mm, TerminalBlock_Phoenix:TerminalBlock_Phoenix_PT-1,5-3-5.0-H_1x03_P5.00mm_Horizontal, F.Cu at (91.0, 108.5)
- added J8: Screw_Terminal_3_P5.00mm, TerminalBlock_Phoenix:TerminalBlock_Phoenix_PT-1,5-3-5.0-H_1x03_P5.00mm_Horizontal, F.Cu at (91.0, 119.8)
- added J9: Screw_Terminal_2_P5.00mm, TerminalBlock_Phoenix:TerminalBlock_Phoenix_PT-1,5-2-5.0-H_1x02_P5.00mm_Horizontal, F.Cu at (108.1, 40.6)
- added K1: G5V-2, Relay_THT:Relay_DPDT_Omron_G5V-2, F.Cu at (145.9, 104.9)
- added Q1: BC548, Package_TO_SOT_THT:TO-92_Inline, F.Cu at (118.6, 121.3)
- added R2: 2.2k, Resistor_THT:R_Axial_DIN0207_L6.3mm_D2.5mm_P10.16mm_Horizontal, F.Cu at (148.2, 41.6)
- added R3: 2.2k, Resistor_THT:R_Axial_DIN0207_L6.3mm_D2.5mm_P10.16mm_Horizontal, F.Cu at (148.2, 45.7)
- added R4: 2.2k, Resistor_THT:R_Axial_DIN0207_L6.3mm_D2.5mm_P10.16mm_Horizontal, F.Cu at (148.2, 49.7)
- added R5: 2.2k, Resistor_THT:R_Axial_DIN0207_L6.3mm_D2.5mm_P10.16mm_Horizontal, F.Cu at (148.2, 53.8)
- added R6: 10k, Resistor_THT:R_Axial_DIN0207_L6.3mm_D2.5mm_P10.16mm_Horizontal, F.Cu at (148.2, 57.8)
- added R7: 10k, Resistor_THT:R_Axial_DIN0207_L6.3mm_D2.5mm_P10.16mm_Horizontal, F.Cu at (148.2, 61.9)
- added R8: 10k, Resistor_THT:R_Axial_DIN0207_L6.3mm_D2.5mm_P10.16mm_Horizontal, F.Cu at (148.2, 65.9)
- added R9: 10k, Resistor_THT:R_Axial_DIN0207_L6.3mm_D2.5mm_P10.16mm_Horizontal, F.Cu at (148.2, 70.0)
- added U3: ESP32-DEVKITC-32D, ESP32-DEVKITC-32D:MODULE_ESP32-DEVKITC-32D, F.Cu at (131.9, 63.5)
- added U4: LM7805_TO220, Package_TO_SOT_THT:TO-220-3_Vertical, F.Cu at (130.6, 122.0)
- added U5: PC817, Package_DIP:DIP-4_W7.62mm, F.Cu at (118.2, 93.6)
- added U6: PC817, Package_DIP:DIP-4_W7.62mm, F.Cu at (118.2, 100.2)
- added U7: PC817, Package_DIP:DIP-4_W7.62mm, F.Cu at (118.2, 106.8)
- added U8: PC817, Package_DIP:DIP-4_W7.62mm, F.Cu at (118.2, 113.5)
- R1: value 0 -> 2.2k; footprint Resistor_SMD:R_0805_2012Metric_Pad1.20x1.40mm_HandSolder -> Resistor_THT:R_Axial_DIN0207_L6.3mm_D2.5mm_P10.16mm_Horizontal
- U2: value TXS0108EPW -> TX0108E-Breakout; footprint Package_SO:TSSOP-20_4.4x6.5mm_P0.65mm -> txs0108e-breakout:txs0108e-breakout
- moved U2 106.0 mm to (135.6, 106.0)
- moved R1 95.8 mm to (148.2, 37.6), turned to 0 degrees
Connections:
- R1 pad 1: VCC -> rele_fiaccola
- R1 pad 2: Net-(P1-P10) -> Net-(Q1-B)
- U2 pad 1: Net-(P1-P2) -> STEP_X_MIC.
- U2 pad 10: Net-(P1-P10) -> GND
- U2 pad 11: GND -> unconnected-(U2-B8-Pad11)
- U2 pad 12: Net-(P2-P9) -> unconnected-(U2-B7-Pad12)
- U2 pad 13: Net-(P2-P8) -> ENABLE_PIN_Y
- U2 pad 14: Net-(P2-P7) -> DIR_PIN_Y
- U2 pad 15: Net-(P2-P6) -> STEP_PIN_Y
- U2 pad 16: Net-(P2-P5) -> ENABLE_PIN_X
- U2 pad 17: Net-(P2-P4) -> DIR_PIN_X
- U2 pad 18: Net-(P2-P3) -> STEP_PIN_X
- U2 pad 19: Net-(P2-P1) -> +5V
- U2 pad 2: VCC -> DIR_X_MIC.
- U2 pad 3: Net-(P1-P3) -> ENBL_X_MIC.
- U2 pad 4: Net-(P1-P4) -> STEP_Y_MIC.
- U2 pad 5: Net-(P1-P5) -> DIR_Y_MIC.
- U2 pad 6: Net-(P1-P6) -> ENBL_Y_MIC.
- U2 pad 7: Net-(P1-P7) -> unconnected-(U2-A7-Pad7)
- U2 pad 8: Net-(P1-P8) -> unconnected-(U2-A8-Pad8)
- U2 pad 9: Net-(P1-P9) -> +3.3V
Routing:
- net Net-(P2-P1): track 39.8 -> 0.00 mm, vias 2 -> 0
- net GND: track 34.1 -> 0.00 mm
- net VCC: track 31.6 -> 0.00 mm
- net Net-(P1-P10): track 28.8 -> 0.00 mm
- net Net-(P1-P9): track 11.1 -> 0.00 mm
- net Net-(P2-P9): track 10.8 -> 0.00 mm
- net Net-(P1-P8): track 9.23 -> 0.00 mm
- net Net-(P2-P8): track 8.94 -> 0.00 mm
- net Net-(P1-P7): track 7.34 -> 0.00 mm
- net Net-(P2-P7): track 7.05 -> 0.00 mm
- net Net-(P1-P2): track 6.44 -> 0.00 mm
- net Net-(P1-P6): track 6.08 -> 0.00 mm
- net Net-(P1-P3): track 5.92 -> 0.00 mm
- net Net-(P2-P2): track 5.81 -> 0.00 mm
- net Net-(P2-P6): track 5.45 -> 0.00 mm
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