File: _autosave-Cordonatrice F.lli Verna.kicad_pcb (KiCad board)
At the start: 2 copper layers, 39 parts, among them J1 Screw_Terminal_3_P5.00mm, J10 Screw_Terminal_2_P5.00mm, J11 Screw_Terminal_2_P5.00mm, J12 Screw_Terminal_4_P5.00mm, J13 Screw_Terminal_2_P5.00mm, J14 Screw_Terminal_2_P5.00mm, J2 Screw_Terminal_3_P5.00mm, J3 Screw_Terminal_3_P5.00mm, J4 Screw_Terminal_3_P5.00mm, J5 Screw_Terminal_3_P5.00mm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

Commit message: aggiunta 7824
Parts:
- removed C1: 22uF_50V, Capacitor_THT:CP_Radial_D5.0mm_P2.00mm
- removed C2: 100nF_Ceramic, Capacitor_THT:C_Disc_D5.0mm_W2.5mm_P2.50mm
- removed U1: LM7812_TO220, Package_TO_SOT_THT:TO-220-3_Vertical
Connections:
- C3 pad 2: Net-(U1-VO) -> +5V
- C6 pad 1: Net-(U1-VO) -> +5V
- U4 pad 1: Net-(U1-VO) -> +24V
