File: Cordonatrice F.lli Verna_mosettirere_piccole.kicad_sch (KiCad schematic)
At the start: 40 parts, among them J1 Screw_Terminal_3_P5.00mm, J10 Screw_Terminal_2_P5.00mm, J11 Screw_Terminal_2_P5.00mm, J12 Screw_Terminal_4_P5.00mm, J13 Screw_Terminal_2_P5.00mm, J14 Screw_Terminal_2_P5.00mm, J2 Screw_Terminal_3_P5.00mm, J3 Screw_Terminal_3_P5.00mm, J4 Screw_Terminal_3_P5.00mm, J5 Screw_Terminal_3_P5.00mm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

Commit message: applicato freerouting
Connections:
- net ENABLE_PIN_X: now also J5.3; no longer J5.1
- net ENABLE_PIN_Y: now also J6.3; no longer J6.1
- net STEP_PIN_X: now also J5.1; no longer J5.3
- net STEP_PIN_Y: now also J6.1; no longer J6.3
Other:
- company: F.lli Verna -> (none)
- title: Cordonatrice automatica  -> (none)
Changed lines of the file:
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@@
 	(generator_version "9.0")
 	(paper "A4")
-	(title_block
-		(title "Cordonatrice automatica ")
-		(date "2025-09-30")
-		(company "F.lli Verna")
-	)
 	(text "Rele"
 		(exclude_from_sim no)
@@
 	(wire
 		(pts
+			(xy 191.77 138.43) (xy 196.85 138.43)
+		)
+		(stroke
+			(width 0)
+			(type default)
+		)
+	)
+	(wire
+		(pts
 			(xy 198.12 34.29) (xy 213.36 34.29)
 		)
@@
 	(wire
 		(pts
-			(xy 191.77 138.43) (xy 198.12 138.43)
+			(xy 85.09 189.23) (xy 85.09 195.58)
 		)
 		(stroke
@@
 	(wire
 		(pts
-			(xy 85.09 189.23) (xy 85.09 195.58)
+			(xy 233.68 100.33) (xy 233.68 96.52)
 		)
 		(stroke
@@
 	(wire
 		(pts
-			(xy 233.68 100.33) (xy 233.68 96.52)
+			(xy 191.77 143.51) (xy 196.85 143.51)
 		)
 		(stroke
@@
 	(wire
 		(pts
-			(xy 191.77 143.51) (xy 199.39 143.51)
-		)
-		(stroke
-			(width 0)
-			(type default)
-		)
-	)
-	(wire
-		(pts
 			(xy 233.68 96.52) (xy 236.22 96.52)
 		)
@@
 	(wire
 		(pts
+			(xy 191.77 156.21) (xy 196.85 156.21)
+		)
+		(stroke
+			(width 0)
+			(type default)
+		)
+	)
+	(wire
+		(pts
 			(xy 38.1 172.72) (xy 38.1 186.69)
 		)
@@
 	(wire
 		(pts
-			(xy 195.58 156.21) (xy 195.58 154.94)
-		)
-		(stroke
-			(width 0)
-			(type default)
-		)
-	)
-	(wire
-		(pts
 			(xy 222.25 96.52) (xy 222.25 99.06)
 		)
@@
 	(wire
 		(pts
-			(xy 191.77 156.21) (xy 195.58 156.21)
-		)
-		(stroke
-			(width 0)
-			(type default)
-		)
-	)
-	(wire
-		(pts
 			(xy 161.29 96.52) (xy 166.37 96.52)
 		)
@@
 	(wire
 		(pts
-			(xy 151.13 107.95) (xy 161.29 107.95)
+			(xy 191.77 161.29) (xy 196.85 161.29)
 		)
 		(stroke
@@
 	(wire
 		(pts
-			(xy 33.02 138.43) (xy 35.56 138.43)
+			(xy 151.13 107.95) (xy 161.29 107.95)
 		)
 		(stroke
@@
 	(wire
 		(pts
-			(xy 151.13 105.41) (xy 151.13 107.95)
+			(xy 33.02 138.43) (xy 35.56 138.43)
 		)
 		(stroke
@@
 	(wire
 		(pts
-			(xy 191.77 161.29) (xy 195.58 161.29)
+			(xy 151.13 105.41) (xy 151.13 107.95)
 		)
 		(stroke
@@
 	(global_label "ENABLE_PIN_Y"
 		(shape input)
-		(at 195.58 156.21 0)
+		(at 196.85 161.29 0)
 		(fields_autoplaced yes)
 		(effects
@@
 		)
 		(property "Intersheetrefs" "${INTERSHEET_REFS}"
-			(at 211.1553 156.21 0)
+			(at 212.4253 161.29 0)
 			(effects
 				(font
@@
 	(global_label "STEP_PIN_X"
 		(shape input)
-		(at 199.39 143.51 0)
+		(at 196.85 138.43 0)
 		(fields_autoplaced yes)
 		(effects
@@
 		)
 		(property "Intersheetrefs" "${INTERSHEET_REFS}"
-			(at 212.6671 143.51 0)
+			(at 210.1271 138.43 0)
 			(effects
 				(font
@@
 	(global_label "STEP_PIN_Y"
 		(shape input)
-		(at 195.58 161.29 0)
+		(at 196.85 156.21 0)
 		(fields_autoplaced yes)
 		(effects
@@
 		)
 		(property "Intersheetrefs" "${INTERSHEET_REFS}"
-			(at 208.7362 161.29 0)
+			(at 210.0062 156.21 0)
 			(effects
 				(font
@@
 	(global_label "ENABLE_PIN_X"
 		(shape input)
-		(at 198.12 138.43 0)
+		(at 196.85 143.51 0)
 		(fields_autoplaced yes)
 		(effects
@@
 		)
 		(property "Intersheetrefs" "${INTERSHEET_REFS}"
-			(at 213.8162 138.43 0)
+			(at 212.5462 143.51 0)
 			(effects
 				(font
